Commit message: Refactoring of cylinder_inertial

File: urdf/inc/ur_common.xacro (robot description, xacro)
@@ -11,8 +11,7 @@
     Contributor: Felix Messmer
   -->
-  <xacro:macro name="cylinder_inertial" params="radius length mass *origin">
+  <xacro:macro name="cylinder_inertial" params="radius length mass origin_xyz:='0 0 0' origin_rpy:='0 0 0'">
     <inertial>
       <mass value="${mass}" />
-      <xacro:insert_block name="origin" />
       <inertia ixx="${0.0833333 * mass * (3 * radius * radius + length * length)}" ixy="0.0" ixz="0.0"
         iyy="${0.0833333 * mass * (3 * radius * radius + length * length)}" iyz="0.0"

File: urdf/ur_macro.xacro (robot description, xacro)
@@ -147,46 +147,32 @@
         </geometry>
       </collision>
-      <xacro:cylinder_inertial radius="${base_inertia_radius}" length="${base_inertia_length}" mass="${base_mass}">
-        <origin xyz="0 0 0" rpy="0 0 0" />
-      </xacro:cylinder_inertial>
+      <xacro:cylinder_inertial radius="${base_inertia_radius}" length="${base_inertia_length}" mass="${base_mass}" />
     </link>
     <xacro:new_link name="shoulder">
       <origin xyz="0 0 0" rpy="0 0 ${pi}"/>
-      <xacro:cylinder_inertial radius="${shoulder_inertia_radius}" length="${shoulder_inertia_length}" mass="${shoulder_mass}">
-        <origin xyz="0 0 0" rpy="0 0 0" />
-      </xacro:cylinder_inertial>
+      <xacro:cylinder_inertial radius="${shoulder_inertia_radius}" length="${shoulder_inertia_length}" mass="${shoulder_mass}" />
     </xacro:new_link>
     <xacro:new_link name="upper_arm">
       <origin xyz="0 0 ${shoulder_offset}" rpy="${pi/2} 0 ${-pi/2}"/>
-      <xacro:cylinder_inertial radius="${upperarm_inertia_radius}" length="${upperarm_inertia_length}" mass="${upper_arm_mass}">
-        <origin xyz="${-0.5 * upperarm_inertia_length} 0.0 ${upper_arm_inertia_offset}" rpy="0 ${pi/2} 0" />
-      </xacro:cylinder_inertial>
+      <xacro:cylinder_inertial radius="${upperarm_inertia_radius}" length="${upperarm_inertia_length}" mass="${upper_arm_mass}" origin_xyz="${-0.5 * upperarm_inertia_length} 0.0 ${upper_arm_inertia_offset}" origin_rpy="0 ${pi/2} 0" />
     </xacro:new_link>
     <xacro:new_link name="forearm">
       <origin xyz="0 0 ${elbow_offset}" rpy="${pi/2} 0 ${-pi/2}"/>
-      <xacro:cylinder_inertial radius="${forearm_inertia_radius}" length="${forearm_inertia_length}"  mass="${forearm_mass}">
-        <origin xyz="${-0.5 * forearm_inertia_length} 0.0 ${elbow_offset}" rpy="0 ${pi/2} 0" />
-      </xacro:cylinder_inertial>
+      <xacro:cylinder_inertial radius="${forearm_inertia_radius}" length="${forearm_inertia_length}"  mass="${forearm_mass}" origin_xyz="${-0.5 * forearm_inertia_length} 0.0 ${elbow_offset}" origin_rpy="0 ${pi/2} 0" />
     </xacro:new_link>
     <xacro:new_link name="wrist_1">
       <xacro:get_visual_params name="wrist_1" type="visual_offset"/>
       <origin xyz="0 0 ${visual_params}" rpy="${pi/2} 0 0"/>
-      <xacro:cylinder_inertial radius="${wrist_1_inertia_radius}" length="${wrist_1_inertia_length}"  mass="${wrist_1_mass}">
-        <origin xyz="0 0 0" rpy="0 0 0" />
-      </xacro:cylinder_inertial>
+      <xacro:cylinder_inertial radius="${wrist_1_inertia_radius}" length="${wrist_1_inertia_length}"  mass="${wrist_1_mass}" />
     </xacro:new_link>
     <xacro:new_link name="wrist_2">
       <xacro:get_visual_params name="wrist_2" type="visual_offset"/>
       <origin xyz="0 0 ${visual_params}" rpy="0 0 0"/>
-      <xacro:cylinder_inertial radius="${wrist_2_inertia_radius}" length="${wrist_2_inertia_length}"  mass="${wrist_2_mass}">
-        <origin xyz="0 0 0" rpy="0 0 0" />
-      </xacro:cylinder_inertial>
+      <xacro:cylinder_inertial radius="${wrist_2_inertia_radius}" length="${wrist_2_inertia_length}"  mass="${wrist_2_mass}" />
     </xacro:new_link>
     <xacro:new_link name="wrist_3">
       <xacro:get_visual_params name="wrist_3" type="visual_offset"/>
       <origin xyz="0 0 ${visual_params}" rpy="${pi/2} 0 0"/>
-      <xacro:cylinder_inertial radius="${wrist_3_inertia_radius}" length="${wrist_3_inertia_length}"  mass="${wrist_3_mass}">
-        <origin xyz="0.0 0.0 ${-0.5 * wrist_3_inertia_length}" rpy="0 0 0" />
-      </xacro:cylinder_inertial>
+      <xacro:cylinder_inertial radius="${wrist_3_inertia_radius}" length="${wrist_3_inertia_length}"  mass="${wrist_3_mass}" origin_xyz="0.0 0.0 ${-0.5 * wrist_3_inertia_length}" />
     </xacro:new_link>
     <!-- base_joint fixes base_link to the environment -->
